File: pcb-hotswap/lancer-hotswap.kicad_pcb (KiCad board)
At the start: 2 copper layers, 209.5 x 76.2 mm, 95 parts, among them SW1 SW_Push, SW10 SW_Push, SW11 SW_Push, SW12 SW_Push, SW13 SW_Push, SW14 SW_Push, SW15 SW_Push, SW16 SW_Push, SW17 SW_Push, SW18 SW_Push, SW19 SW_Push, SW2 SW_Push, SW20 SW_Push, SW21 SW_Push, SW22 SW_Push, SW23 SW_Push, SW24 SW_Push, SW25 SW_Push, SW26 SW_Push, SW27 SW_Push, SW28 SW_Push, SW29 SW_Push, SW3 SW_Push, SW30 SW_Push, SW31 SW_Push, SW32 SW_Push, SW33 SW_Push, SW34 SW_Push, SW35 SW_Push, SW36 SW_Push, SW37 SW_SPDT, SW38 SW_Push, SW4 SW_Push, SW5 SW_Push, SW6 SW_Push, SW7 SW_Push, SW8 SW_Push, SW9 SW_Push, U1 ProMicro_Flipped

Commit message: v1.1
Parts:
- added REF**: On, lancer:On, F.Cu at (128.9, 22.2)
- added REF**: Off, lancer:Off, F.Cu at (122.6, 22.2)
- moved D31 10.2 mm to (78.1, 82.5)
- moved D32 10.2 mm to (97.2, 82.5)
- moved D33 10.2 mm to (116.2, 82.5)
- moved D34 10.2 mm to (135.3, 82.5)
- moved D35 10.2 mm to (154.3, 82.5)
- moved D36 10.2 mm to (173.4, 82.5)
- moved O1 1.27 mm to (125.7, 58.4)
- turned SW31 to 180 degrees
- turned SW32 to 180 degrees
- turned SW33 to 180 degrees
- turned SW34 to 180 degrees
- turned SW35 to 180 degrees
- turned SW36 to 180 degrees
Connections:
- D31 pad 2: Net-(D31-Pad2) -> Net-(D31-A)
- D32 pad 2: Net-(D32-Pad2) -> Net-(D32-A)
- D33 pad 2: Net-(D33-Pad2) -> Net-(D33-A)
- D34 pad 2: Net-(D34-Pad2) -> Net-(D34-A)
- D35 pad 2: Net-(D35-Pad2) -> Net-(D35-A)
- D36 pad 2: Net-(D36-Pad2) -> Net-(D36-A)
- SW31 pad 1: Net-(D31-Pad2) -> /C2
- SW31 pad 2: /C2 -> Net-(D31-A)
- SW32 pad 1: Net-(D32-Pad2) -> /C3
- SW32 pad 2: /C3 -> Net-(D32-A)
- SW33 pad 1: Net-(D33-Pad2) -> /C4
- SW33 pad 2: /C4 -> Net-(D33-A)
- SW34 pad 1: /C5 -> Net-(D34-A)
- SW34 pad 2: Net-(D34-Pad2) -> /C5
- SW35 pad 1: /C6 -> Net-(D35-A)
- SW35 pad 2: Net-(D35-Pad2) -> /C6
- SW36 pad 1: /C7 -> Net-(D36-A)
- SW36 pad 2: Net-(D36-Pad2) -> /C7
Routing:
- net /R4: track 147.7 -> 131.9 mm, vias 8 -> 7
- net Net-(D35-Pad2): track 14.5 -> 0.00 mm
- net Net-(D36-Pad2): track 14.5 -> 0.00 mm
- net Net-(D34-Pad2): track 14.5 -> 0.00 mm
- net Net-(D33-A): track 0.00 -> 13.6 mm
- net Net-(D32-A): track 0.00 -> 13.6 mm
- net Net-(D31-A): track 0.00 -> 13.6 mm
- net Net-(D33-Pad2): track 11.8 -> 0.00 mm
- net Net-(D32-Pad2): track 11.8 -> 0.00 mm
- net Net-(D31-Pad2): track 11.8 -> 0.00 mm
- net Net-(D36-A): track 0.00 -> 11.4 mm
- net Net-(D34-A): track 0.00 -> 11.4 mm
- net Net-(D35-A): track 0.00 -> 11.4 mm
- net /C4: track 67.9 -> 76.0 mm
- net /C3: track 92.3 -> 100.5 mm
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