File: pcb-hotswap/lancer-hotswap.kicad_sch (KiCad schematic)
At the start: 88 parts, among them SW1 SW_Push, SW10 SW_Push, SW11 SW_Push, SW12 SW_Push, SW13 SW_Push, SW14 SW_Push, SW15 SW_Push, SW16 SW_Push, SW17 SW_Push, SW18 SW_Push, SW19 SW_Push, SW2 SW_Push, SW20 SW_Push, SW21 SW_Push, SW22 SW_Push, SW23 SW_Push, SW24 SW_Push, SW25 SW_Push, SW26 SW_Push, SW27 SW_Push, SW28 SW_Push, SW29 SW_Push, SW3 SW_Push, SW30 SW_Push, SW31 SW_Push, SW32 SW_Push, SW33 SW_Push, SW34 SW_Push, SW35 SW_Push, SW36 SW_Push, SW37 SW_SPDT, SW38 SW_Push, SW4 SW_Push, SW5 SW_Push, SW6 SW_Push, SW7 SW_Push, SW8 SW_Push, SW9 SW_Push, U1 ProMicro_Flipped

Commit message: v1.1
Connections:
- net C2: now also SW31.1; no longer SW31.2
- net C3: now also SW32.1; no longer SW32.2
- net C4: now also SW33.1; no longer SW33.2
- net C5: now also SW34.2; no longer SW34.1
- net C6: now also SW35.2; no longer SW35.1
- net C7: now also SW36.2; no longer SW36.1
- net at D36.2 (A): now also SW36.1; no longer SW36.2
- net at D32.2 (A): now also SW32.2; no longer SW32.1
- net at D34.2 (A): now also SW34.1; no longer SW34.2
- net at D33.2 (A): now also SW33.2; no longer SW33.1
- net at D35.2 (A): now also SW35.1; no longer SW35.2
- net at D31.2 (A): now also SW31.2; no longer SW31.1
Other:
- moved on the sheet: SW31, SW32, SW33, SW34, SW35, SW36
